File: esp8266/idf/proyectos/iotTermometro/kicad/usb/usb.kicad_sch (KiCad schematic)
At the start: 12 parts, among them J1 USB_A, SW1 SW_Push, U1 AMS1117-3.3, U2 ESP-12F, U3 DS18B20

Commit message: x
Parts:
- removed J1: USB_A, Connector_USB:USB_A_CNCTech_1001-011-01101_Horizontal, symbol Connector:USB_A
- added J1: USB-AM-S-X-X-TH, conector_usb:SAMTEC_USB-AM-S-X-X-TH, symbol USB-AM-S-X-X-TH:USB-AM-S-X-X-TH
Connections:
- net GND: now also J1.04 (GND)
- net RX: now also J1.02 (D-)
- net TX: now also J1.03 (D+)
- net VIN: now also J1.01 (VCC)
- new net: J1.S1 (SHIELD), J1.S2 (SHIELD)
Changed lines of the file:
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@@
   (junction (at 177.8 58.42) (diameter 0) (color 0 0 0 0)
   )
+  (no_connect (at 222.25 68.58))
   (no_connect (at 147.32 92.71))
-  (no_connect (at 217.17 104.14))
   (no_connect (at 147.32 107.95))
   (no_connect (at 147.32 105.41))
@@
     (stroke (width 0) (type default) (color 0 0 0 0))
   )
+  (label "RX" (at 222.25 58.42 180)
+    (effects (font (size 1.27 1.27)) (justify right bottom))
+  )
   (label "LED_FUNCION" (at 190.5 120.65 180)
     (effects (font (size 1.27 1.27)) (justify right bottom))
@@
     (effects (font (size 1.27 1.27)) (justify right bottom))
   )
-  (label "VIN" (at 227.33 88.9 0)
-    (effects (font (size 1.27 1.27)) (justify left bottom))
-  )
   (label "NET_BOTON" (at 147.32 82.55 0)
     (effects (font (size 1.27 1.27)) (justify left bottom))
@@
     (effects (font (size 1.27 1.27)) (justify left bottom))
   )
-  (label "TX" (at 227.33 93.98 0)
-    (effects (font (size 1.27 1.27)) (justify left bottom))
-  )
-  (label "RX" (at 227.33 96.52 0)
-    (effects (font (size 1.27 1.27)) (justify left bottom))
-  )
   (label "NET_BOTON" (at 175.26 60.96 180)
     (effects (font (size 1.27 1.27)) (justify right bottom))
@@
     (effects (font (size 1.27 1.27)) (justify left bottom))
   )
+  (label "TX" (at 222.25 60.96 180)
+    (effects (font (size 1.27 1.27)) (justify right bottom))
+  )
   (label "VCC" (at 177.8 41.91 180)
+    (effects (font (size 1.27 1.27)) (justify right bottom))
+  )
+  (label "VIN" (at 222.25 55.88 180)
     (effects (font (size 1.27 1.27)) (justify right bottom))
   )
@@
     (pin "2")
   )
-  (symbol (lib_id "power:GND") (at 219.71 104.14 0) (unit 1)
-    (in_bom yes) (on_board yes) (fields_autoplaced)
-    (property "Reference" "#PWR09" (id 0) (at 219.71 110.49 0)
-      (effects (font (size 1.27 1.27)) hide)
-    )
-    (property "Value" "GND" (id 1) (at 219.71 109.22 0))
-    (property "Footprint" "" (id 2) (at 219.71 104.14 0)
-      (effects (font (size 1.27 1.27)) hide)
-    )
-    (property "Datasheet" "" (id 3) (at 219.71 104.14 0)
-      (effects (font (size 1.27 1.27)) hide)
-    )
-    (pin "1")
-  )
   (symbol (lib_id "Regulator_Linear:AMS1117-3.3") (at 87.63 49.53 0) (unit 1)
     (in_bom yes) (on_board yes) (fields_autoplaced)
@@
     (pin "2")
   )
+  (symbol (lib_id "USB-AM-S-X-X-TH:USB-AM-S-X-X-TH") (at 232.41 60.96 0) (unit 1)
+    (in_bom yes) (on_board yes) (fields_autoplaced)
+    (property "Reference" "J1" (id 0) (at 238.76 60.9599 0)
+      (effects (font (size 1.27 1.27)) (justify left))
+    )
+    (property "Value" "USB-AM-S-X-X-TH" (id 1) (at 238.76 63.4999 0)
+      (effects (font (size 1.27 1.27)) (justify left))
+    )
+    (property "Footprint" "conector_usb:SAMTEC_USB-AM-S-X-X-TH" (id 2) (at 232.41 60.96 0)
+      (effects (font (size 1.27 1.27)) (justify left bottom) hide)
+    )
+    (property "Datasheet" "" (id 3) (at 232.41 60.96 0)
+      (effects (font (size 1.27 1.27)) (justify left bottom) hide)
+    )
+    (property "STANDARD" "Manufacturer Recommendations" (id 4) (at 232.41 60.96 0)
+      (effects (font (size 1.27 1.27)) (justify left bottom) hide)
+    )
+    (property "MAXIMUM_PACKAGE_HEIGHT" "4.6 mm" (id 5) (at 232.41 60.96 0)
+      (effects (font (size 1.27 1.27)) (justify left bottom) hide)
+    )
+    (property "MANUFACTURER" "Samtec" (id 6) (at 232.41 60.96 0)
+      (effects (font (size 1.27 1.27)) (justify left bottom) hide)
+    )
+    (property "PARTREV" "U" (id 7) (at 232.41 60.96 0)
+      (effects (font (size 1.27 1.27)) (justify left bottom) hide)
+    )
+    (pin "01")
+    (pin "02")
+    (pin "03")
+    (pin "04")
+    (pin "S1")
+    (pin "S2")
+  )
   (symbol (lib_id "power:GND") (at 71.12 58.42 0) (unit 1)
     (in_bom yes) (on_board yes) (fields_autoplaced)
@@
     )
     (property "Datasheet" "" (id 3) (at 205.74 120.65 0)
+      (effects (font (size 1.27 1.27)) hide)
+    )
+    (pin "1")
+  )
+  (symbol (lib_id "power:GND") (at 222.25 63.5 270) (unit 1)
+    (in_bom yes) (on_board yes) (fields_autoplaced)
+    (property "Reference" "#PWR08" (id 0) (at 215.9 63.5 0)
+      (effects (font (size 1.27 1.27)) hide)
+    )
+    (property "Value" "GND" (id 1) (at 217.17 63.5 0))
+    (property "Footprint" "" (id 2) (at 222.25 63.5 0)
+      (effects (font (size 1.27 1.27)) hide)
+    )
+    (property "Datasheet" "" (id 3) (at 222.25 63.5 0)
       (effects (font (size 1.27 1.27)) hide)
     )
@@
     (pin "2")
     (pin "3")
-  )
-  (symbol (lib_id "Connector:USB_A") (at 219.71 93.98 0) (unit 1)
-    (in_bom yes) (on_board yes) (fields_autoplaced)
-    (property "Reference" "J1" (id 0) (at 219.71 81.28 0))
-    (property "Value" "USB_A" (id 1) (at 219.71 83.82 0))
-    (property "Footprint" "Connector_USB:USB_A_CNCTech_1001-011-01101_Horizontal" (id 2) (at 223.52 95.25 0)
-      (effects (font (size 1.27 1.27)) hide)
-    )
-    (property "Datasheet" " ~" (id 3) (at 223.52 95.25 0)
-      (effects (font (size 1.27 1.27)) hide)
-    )
-    (pin "1")
-    (pin "2")
-    (pin "3")
-    (pin "4")
-    (pin "5")
   )
   (symbol (lib_id "Device:C_Polarized") (at 104.14 54.61 0) (unit 1)
@@
       (reference "#PWR07") (unit 1) (value "GND") (footprint "")
     )
-    (path "/1339f491-7586-475c-a3ec-3f3fa1db9183"
-      (reference "#PWR09") (unit 1) (value "GND") (footprint "")
+    (path "/57ea5df2-8327-4992-82c1-92a678724bbb"
+      (reference "#PWR08") (unit 1) (value "GND") (footprint "")
     )
     (path "/edf6191d-434c-40ac-a287-ce0b6f906e77"
@@
       (reference "D1") (unit 1) (value "LED") (footprint "LED_SMD:LED_0603_1608Metric")
     )
-    (path "/d87cc3e6-70e4-41ba-bfa9-1612995ab3dd"
-      (reference "J1") (unit 1) (value "USB_A") (footprint "Connector_USB:USB_A_CNCTech_1001-011-01101_Horizontal")
+    (path "/4117bdfe-60ca-4f2c-8585-3d6821fc99e1"
+      (reference "J1") (unit 1) (value "USB-AM-S-X-X-TH") (footprint "conector_usb:SAMTEC_USB-AM-S-X-X-TH")
     )
     (path "/3d22e2d7-fcae-45b0-aa99-f847037dbf41"
