File: esp8266/idf/proyectos/iotOnOff/kicad/dinrail/iotOnOff.kicad_sch (KiCad schematic)
At the start: 21 parts, among them J1 Conn_01x02, J2 Conn_01x02, J3 Conn_01x04, K1 SANYOU_SRD_Form_A, Q1 2N7002, SW1 SW_Push, U1 AMS1117-3.3, U3 ESP-12F

Commit message: Se corrige la conexion de GPIO15 en dinrail
Parts:
- R6, RV1, RV2: footprint (none) -> Resistor_THT:R_Axial_DIN0411_L9.9mm_D3.6mm_P7.62mm_Vertical
Connections:
- net GND: now also U3.16 (GPIO15)
- net at U3.17 (GPIO2): no longer U3.16 (GPIO15)
- no-connect marks 12 -> 13
Changed lines of the file:
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@@
   (no_connect (at 122.6058 119.8118))
   (no_connect (at 153.0858 112.1918))
+  (no_connect (at 153.0858 96.9518))
   (no_connect (at 122.6058 102.0318))
   (no_connect (at 122.6058 91.8718))
@@
     (stroke (width 0) (type default) (color 0 0 0 0))
   )
+  (wire (pts (xy 153.0858 114.7318) (xy 157.2 114.7318))
+    (stroke (width 0) (type default) (color 0 0 0 0))
+  )
   (wire (pts (xy 105.5624 79.4004) (xy 157.1752 79.4004))
     (stroke (width 0) (type default) (color 0 0 0 0))
   )
-  (wire (pts (xy 153.0858 114.7318) (xy 155.5 114.7318))
-    (stroke (width 0) (type default) (color 0 0 0 0))
-  )
   (wire (pts (xy 71.8566 51.2318) (xy 74.0521 51.2318))
     (stroke (width 0) (type default) (color 0 0 0 0))
@@
     (stroke (width 0) (type default) (color 0 0 0 0))
   )
+  (wire (pts (xy 157.2 114.7318) (xy 157.2 114.9))
+    (stroke (width 0) (type default) (color 0 0 0 0))
+  )
   (wire (pts (xy 117.1702 89.916) (xy 117.1702 96.9518))
     (stroke (width 0) (type default) (color 0 0 0 0))
   )
-  (wire (pts (xy 155.5 96.9518) (xy 153.0858 96.9518))
-    (stroke (width 0) (type default) (color 0 0 0 0))
-  )
   (wire (pts (xy 45.3136 110.1344) (xy 74.0521 110.1344))
     (stroke (width 0) (type default) (color 0 0 0 0))
@@
   )
   (wire (pts (xy 254.9398 95.5294) (xy 257.7592 95.5294))
-    (stroke (width 0) (type default) (color 0 0 0 0))
-  )
-  (wire (pts (xy 155.5 114.7318) (xy 155.5 96.9518))
     (stroke (width 0) (type default) (color 0 0 0 0))
   )
@@
     (pin "2")
   )
+  (symbol (lib_id "power:GND") (at 157.2 114.9 0) (unit 1)
+    (in_bom yes) (on_board yes) (fields_autoplaced)
+    (property "Reference" "#PWR0108" (id 0) (at 157.2 121.25 0)
+      (effects (font (size 1.27 1.27)) hide)
+    )
+    (property "Value" "" (id 1) (at 157.2 119.53 0))
+    (property "Footprint" "" (id 2) (at 157.2 114.9 0)
+      (effects (font (size 1.27 1.27)) hide)
+    )
+    (property "Datasheet" "" (id 3) (at 157.2 114.9 0)
+      (effects (font (size 1.27 1.27)) hide)
+    )
+    (pin "1")
+  )
   (symbol (lib_id "Device:Varistor") (at 241.9 118.7 0) (unit 1)
     (in_bom yes) (on_board yes) (fields_autoplaced)
@@
       (effects (font (size 1.27 1.27)) (justify left))
     )
-    (property "Footprint" "" (id 2) (at 240.122 118.7 90)
+    (property "Footprint" "Resistor_THT:R_Axial_DIN0411_L9.9mm_D3.6mm_P7.62mm_Vertical" (id 2) (at 240.122 118.7 90)
       (effects (font (size 1.27 1.27)) hide)
     )
@@
       (effects (font (size 1.27 1.27)) (justify left))
     )
-    (property "Footprint" "" (id 2) (at 47.022 55.9 90)
+    (property "Footprint" "Resistor_THT:R_Axial_DIN0411_L9.9mm_D3.6mm_P7.62mm_Vertical" (id 2) (at 47.022 55.9 90)
       (effects (font (size 1.27 1.27)) hide)
     )
@@
     (property "Reference" "R6" (id 0) (at 41.0412 53.34 90))
     (property "Value" "10" (id 1) (at 41.0412 55.88 90))
-    (property "Footprint" "" (id 2) (at 41.0412 61.4706 90)
+    (property "Footprint" "Resistor_THT:R_Axial_DIN0411_L9.9mm_D3.6mm_P7.62mm_Vertical" (id 2) (at 41.0412 61.4706 90)
       (effects (font (size 1.27 1.27)) hide)
     )
@@
       (reference "#PWR0107") (unit 1) (value "GND") (footprint "")
     )
+    (path "/0723f6ef-563d-44b0-8028-0c69a74665bc"
+      (reference "#PWR0108") (unit 1) (value "GND") (footprint "")
+    )
     (path "/00000000-0000-0000-0000-0000601f810e"
